Commit message: Made URDFs ingestable by regular ROS tools.

File: mhs/MHS.urdf (robot description, URDF)
Before this commit: robot , 13 links, 12 joints
Links:
- link Body_MHS_BottomBlades_v16: geometry visual mesh filename=package://m2020_description/mhs/meshes/MHS_BottomBlades_v16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 scale=1 1 1
- link Body_MHS_Leg01_v16: geometry visual mesh filename=package://m2020_description/mhs/meshes/MHS_Leg01_v16.glb scale=1 1 1
- link Body_MHS_Leg02_v16: geometry visual mesh filename=package://m2020_description/mhs/meshes/MHS_Leg02_v16.glb scale=1 1 1
- link Body_MHS_Leg03_v16: geometry visual mesh filename=package://m2020_description/mhs/meshes/MHS_Leg03_v16.glb scale=1 1 1
- link Body_MHS_Leg04_v16: geometry visual mesh filename=package://m2020_description/mhs/meshes/MHS_Leg04_v16.glb scale=1 1 1
- link Body_MHS_MainBody_v16: geometry visual mesh filename=package://m2020_description/mhs/meshes/MHS_MainBody_v16.glb scale=1 1 1
- link Body_MHS_TopBlades_v16: geometry visual mesh filename=package://m2020_description/mhs/meshes/MHS_TopBlades_v16.glb scale=1 1 1
Joints:
- joint Joint_Leg01_Axis: limit lower=-1.79769e+308 upper=1.79769e+308 effort=1.79769e+308 velocity=1.79769e+308 -> lower=-0.785 upper=0.785 effort=6.28 velocity=6.28
- joint Joint_Leg02_Axis: limit lower=-1.79769e+308 upper=1.79769e+308 effort=1.79769e+308 velocity=1.79769e+308 -> lower=-0.785 upper=0.785 effort=6.28 velocity=6.28
- joint Joint_Leg03_Axis: limit lower=-1.79769e+308 upper=1.79769e+308 effort=1.79769e+308 velocity=1.79769e+308 -> lower=-0.785 upper=0.785 effort=6.28 velocity=6.28
- joint Joint_Leg04_Axis: limit lower=-1.79769e+308 upper=1.79769e+308 effort=1.79769e+308 velocity=1.79769e+308 -> lower=-0.785 upper=0.785 effort=6.28 velocity=6.28
- joint MHS_BottomBlades_v16: limit lower=-1.79769e+308 upper=1.79769e+308 effort=1.79769e+308 velocity=1.79769e+308 -> (none); type revolute -> continuous
- joint MHS_NAVCAM: type None -> fixed
- joint MHS_TopBlades_v16: limit lower=-1.79769e+308 upper=1.79769e+308 effort=1.79769e+308 velocity=1.79769e+308 -> (none); type revolute -> continuous

File: rover/m2020.urdf (robot description, URDF)
Before this commit: robot Perseverance, 115 links, 114 joints
Links:
- link Body_BogieLeft: geometry visual mesh filename=package://m2020_description/rover/meshes/Left_Bogie.gltf scale=1 1 1
- link Body_BogieRight: geometry visual mesh filename=package://m2020_description/rover/meshes/Right_Bogie.gltf scale=1 1 1
- link Body_Chassis: geometry visual mesh filename=package://m2020_description/rover/meshes/CHASSIS.gltf scale=1 1 1
- link Body_CorerFeed: geometry visual mesh filename=package://m2020_description/rover/meshes/AbradingBitInTurre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 scale=1 1 1
- link Body_Differential: geometry visual mesh filename=package://m2020_description/rover/meshes/CenterDifferential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 scale=1 1 1
- link Body_HGA_AZ: geometry visual mesh filename=package://m2020_description/rover/meshes/HGA_AZ.gltf scale=1 1 1
- link Body_HGA_EL: geometry visual mesh filename=package://m2020_description/rover/meshes/HGA_EL.gltf scale=1 1 1
- link Body_RA_Link1: geometry visual mesh filename=package://m2020_description/rover/meshes/Arm_LINK_1.gltf scale=1 1 1
- link Body_RA_Link2: geometry visual mesh filename=package://m2020_description/rover/meshes/Arm_LINK_2.gltf scale=1 1 1
- link Body_RA_Link3: geometry visual mesh filename=package://m2020_description/rover/meshes/Arm_LINK_3.gltf scale=1 1 1
- link Body_RA_Link4: geometry visual mesh filename=package://m2020_description/rover/meshes/Arm_LINK_4.gltf scale=1 1 1
- link Body_RA_Link5: geometry visual mesh filename=package://m2020_description/rover/meshes/Arm_LINK_5.gltf scale=1 1 1
- link Body_RSM_AZ: geometry visual mesh filename=package://m2020_description/rover/meshes/RSM.gltf scale=1 1 1
- link Body_RSM_EL: geometry visual mesh filename=package://m2020_description/rover/meshes/RSM_Head.gltf scale=1 1 1
- link Body_RockerLeft: geometry visual mesh filename=package://m2020_description/rover/meshes/Left_Rocker.gltf scale=1 1 1
- link Body_RockerRight: geometry visual mesh filename=package://m2020_description/rover/meshes/Right_Rocker.gltf scale=1 1 1
- link Body_SHERLOC_Cap: geometry visual mesh filename=package://m2020_description/rover/meshes/ContextImager_Cap.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 scale=1 1 1
- link Body_StabilizerFar: geometry visual mesh filename=package://m2020_description/rover/meshes/StabilizerFarInTur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 scale=1 1 1
- link Body_StabilizerNear: geometry visual mesh filename=package://m2020_description/rover/meshes/StabilizerNearInTu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 scale=1 1 1
- link Body_SteerLeftFront: geometry visual mesh filename=package://m2020_description/rover/meshes/Steer_LeftFront.gl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 scale=1 1 1
- link Body_SteerLeftRear: geometry visual mesh filename=package://m2020_description/rover/meshes/Steer_LeftRear.gltf scale=1 1 1
- link Body_SteerRightFront: geometry visual mesh filename=package://m2020_description/rover/meshes/Steer_RightFront.g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 scale=1 1 1
- link Body_SteerRightRear: geometry visual mesh filename=package://m2020_description/rover/meshes/Steer_RightRear.gl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 scale=1 1 1
- link Body_Turret: geometry visual mesh filename=package://m2020_description/rover/meshes/Turret.gltf scale=1 1 1
- link Body_WATSON_Cap: geometry visual mesh filename=package://m2020_description/rover/meshes/WATSON_Camera_Cap.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 scale=1 1 1
- link Body_WheelLeftFront: geometry visual mesh filename=package://m2020_description/rover/meshes/Wheel_LeftFront.gl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 scale=1 1 1
- link Body_WheelLeftMiddle: geometry visual mesh filename=package://m2020_description/rover/meshes/Wheel_LeftMiddle.g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 scale=1 1 1
- link Body_WheelLeftRear: geometry visual mesh filename=package://m2020_description/rover/meshes/Wheel_LeftRear.gltf scale=1 1 1
- link Body_WheelRightFront: geometry visual mesh filename=package://m2020_description/rover/meshes/Wheel_RightFront.g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 scale=1 1 1
- link Body_WheelRightMiddle: geometry visual mesh filename=package://m2020_description/rover/meshes/Wheel_RightMiddle.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 scale=1 1 1
- link Body_WheelRightRear: geometry visual mesh filename=package://m2020_description/rover/meshes/Wheel_RightRear.gl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 scale=1 1 1
Joints:
- joint CENTER_DIFFERENTIAL: limit lower=-1.79769e+308 upper=1.79769e+308 effort=1.79769e+308 velocity=1.79769e+308 -> lower=-0.225 upper=0.225 effort=6.28 velocity=6.28
- joint DRILL_FEED: limit lower=-1.79769e+308 upper=1.79769e+308 effort=1.79769e+308 velocity=1.79769e+308 -> lower=0.0 upper=0.1 effort=6.28 velocity=6.28
- joint HGA_AZ: limit lower=-1.79769e+308 upper=1.79769e+308 effort=1.79769e+308 velocity=1.79769e+308 -> lower=-0.785 upper=0.785 effort=6.28 velocity=6.28
- joint HGA_EL: limit lower=-1.79769e+308 upper=1.79769e+308 effort=1.79769e+308 velocity=1.79769e+308 -> lower=-0.785 upper=0.785 effort=6.28 velocity=6.28
- joint JOINT1_ENC: limit lower=-3.145 upper=1.592 effort=1.79769e+308 velocity=1.79769e+308 -> lower=-3.145 upper=1.592 effort=6.28 velocity=6.28
- joint JOINT2_ENC: limit lower=-3.267 upper=0.126 effort=1.79769e+308 velocity=1.79769e+308 -> lower=-3.267 upper=0.126 effort=6.28 velocity=6.28
- joint JOINT3_ENC: limit lower=-2.866 upper=2.866 effort=1.79769e+308 velocity=1.79769e+308 -> lower=-2.866 upper=2.866 effort=6.28 velocity=6.28
- joint JOINT4_ENC: limit lower=-0.178 upper=3.669 effort=1.79769e+308 velocity=1.79769e+308 -> lower=-0.178 upper=3.669 effort=6.28 velocity=6.28
- joint JOINT5_ENC: limit lower=-0.353 upper=6.636 effort=1.79769e+308 velocity=1.79769e+308 -> lower=-0.353 upper=6.636 effort=6.28 velocity=6.28
- joint LEFT_BOGIE: limit lower=-1.79769e+308 upper=1.79769e+308 effort=1.79769e+308 velocity=1.79769e+308 -> lower=-0.785 upper=0.785 effort=6.28 velocity=6.28
- joint LEFT_DIFFERENTIAL: limit lower=-1.79769e+308 upper=1.79769e+308 effort=1.79769e+308 velocity=1.79769e+308 -> lower=-0.785 upper=0.785 effort=6.28 velocity=6.28
- joint LF_DRIVE: limit lower=-1.79769e+308 upper=1.79769e+308 effort=1.79769e+308 velocity=1.79769e+308 -> effort=6.28 velocity=6.28; type revolute -> continuous
- joint LF_STEER: limit lower=-1.79769e+308 upper=1.79769e+308 effort=1.79769e+308 velocity=1.79769e+308 -> lower=-3.14 upper=3.14 effort=6.28 velocity=6.28
- joint LM_DRIVE: limit lower=-1.79769e+308 upper=1.79769e+308 effort=1.79769e+308 velocity=1.79769e+308 -> effort=6.28 velocity=6.28; type revolute -> continuous
- joint LR_DRIVE: limit lower=-1.79769e+308 upper=1.79769e+308 effort=1.79769e+308 velocity=1.79769e+308 -> effort=6.28 velocity=6.28; type revolute -> continuous
- joint LR_STEER: limit lower=-1.79769e+308 upper=1.79769e+308 effort=1.79769e+308 velocity=1.79769e+308 -> lower=-3.14 upper=3.14 effort=6.28 velocity=6.28
- joint RF_DRIVE: limit lower=-1.79769e+308 upper=1.79769e+308 effort=1.79769e+308 velocity=1.79769e+308 -> effort=6.28 velocity=6.28; type revolute -> continuous
- joint RF_STEER: limit lower=-1.79769e+308 upper=1.79769e+308 effort=1.79769e+308 velocity=1.79769e+308 -> lower=-3.14 upper=3.14 effort=6.28 velocity=6.28
- joint RIGHT_BOGIE: limit lower=-1.79769e+308 upper=1.79769e+308 effort=1.79769e+308 velocity=1.79769e+308 -> lower=-0.785 upper=0.785 effort=6.28 velocity=6.28
- joint RIGHT_DIFFERENTIAL: limit lower=-1.79769e+308 upper=1.79769e+308 effort=1.79769e+308 velocity=1.79769e+308 -> lower=-0.785 upper=0.785 effort=6.28 velocity=6.28
- joint RM_DRIVE: limit lower=-1.79769e+308 upper=1.79769e+308 effort=1.79769e+308 velocity=1.79769e+308 -> effort=6.28 velocity=6.28; type revolute -> continuous
- joint RR_DRIVE: limit lower=-1.79769e+308 upper=1.79769e+308 effort=1.79769e+308 velocity=1.79769e+308 -> effort=6.28 velocity=6.28; type revolute -> continuous
- joint RR_STEER: limit lower=-1.79769e+308 upper=1.79769e+308 effort=1.79769e+308 velocity=1.79769e+308 -> lower=-3.14 upper=3.14 effort=6.28 velocity=6.28
- joint RSM_AZ_ENC: limit lower=0 upper=6.31809 effort=1.79769e+308 velocity=1.79769e+308 -> lower=0 upper=6.31809 effort=6.28 velocity=6.28
- joint RSM_EL_ENC: limit lower=0 upper=3.1765 effort=1.79769e+308 velocity=1.79769e+308 -> lower=0 upper=3.1765 effort=6.28 velocity=6.28
- joint SHERLOC_CAP_ENC: limit lower=-1.79769e+308 upper=1.79769e+308 effort=1.79769e+308 velocity=1.79769e+308 -> lower=0 upper=1.57 effort=6.28 velocity=6.28
- joint STABILIZER_LOWER: limit lower=-1.79769e+308 upper=1.79769e+308 effort=1.79769e+308 velocity=1.79769e+308 -> lower=-0.5 upper=0.0 effort=6.28 velocity=6.28
- joint STABILIZER_UPPER: limit lower=-1.79769e+308 upper=1.79769e+308 effort=1.79769e+308 velocity=1.79769e+308 -> lower=-0.5 upper=0.0 effort=6.28 velocity=6.28
- joint WATSON_CAP_ENC: limit lower=-1.79769e+308 upper=1.79769e+308 effort=1.79769e+308 velocity=1.79769e+308 -> lower=0.0 upper=1.57 effort=6.28 velocity=6.28
